File: pcb/ReplicaDriverPuenteHL298.kicad_pcb (KiCad board)
At the start: 2 copper layers, 50 x 50 mm, 29 parts, among them J1 Conn_01x04, J2 Conn_01x02, J3 Conn_01x02, J4 Conn_01x02, J5 Conn_01x02, J6 Conn_01x02, J7 Conn_01x03, U1 L298HN, U2 LM78M05

Commit message: Add files via upload
Routing:
- added copper zone on F.Cu, net GND

Commit message: Add files via upload
Other:
- board text added: "0,4 mm;"
- board text added: "1 mm; 0.8 mm;"
- board text added: "1 oz"
- board text added: "Core 1,6 mm"
- board text added: "Diseñado en Argentina"
- board text added: "Dist. a borde: 0,5 mm"
- board text added: "Especificaciones técnicas"
- board text added: "Fabricante: Ernesto Meyer"
- board text added: "Grillas: 0,5 mm; 0,25 mm"
- board text added: "Margen: 0,4 mm"
- board text added: "Pista: 2,5 mm; 2,1 mm;"
- board text added: "SIG B. Cu"
- board text added: "SIG F. Cu"
- board text added: "Terminación: Estaño-Plomo(Sn/Pb)"
- board text added: "Vias: 1,6 mm/0,8 mm; 0,7 mm/0,4 mm"
Changed lines of the file:
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@@
   (general
     (thickness 1.6)
-    (drawings 16)
+    (drawings 38)
     (tracks 162)
     (zones 0)
@@
   (page A4)
   (title_block
+    (title ReplicaDriverPuenteHL298)
+    (date 2021-10-13)
+    (rev 1.0)
     (comment 1 "Diseño bajo licencia CERN-OHL-P.")
+    (comment 2 "Autor: Damián Caputo")
   )
   (layers
@@
     (pad_to_mask_clearance 0)
     (aux_axis_origin 0 0)
+    (grid_origin 125.5 121)
     (visible_elements 7FFFFFFF)
     (pcbplotparams
@@
       (outputformat 1)
       (mirror false)
-      (drillshape 1)
+      (drillshape 0)
       (scaleselection 1)
       (outputdirectory ""))
@@
     )
   )
-  (gr_text "ReplicaDriverPuenteHL298\nCESE2021\nIng.DamianCaputo" (at 150.5 75) (layer B.Mask)
+  (gr_text "Diseñado en Argentina" (at 128.5 89 90) (layer B.SilkS)
+    (effects (font (size 1 1) (thickness 0.15)) (justify mirror))
+  )
+  (gr_line (start 125.5 71) (end 175.5 71) (layer Edge.Cuts) (width 0.2))
+  (gr_text "Fabricante: Ernesto Meyer" (at 220 107) (layer Dwgs.User)
+    (effects (font (size 2 2) (thickness 0.2)))
+  )
+  (gr_text "1 oz" (at 247.5 125.5) (layer Dwgs.User)
+    (effects (font (size 2 2) (thickness 0.2)))
+  )
+  (gr_text "1 oz" (at 247.5 120) (layer Dwgs.User)
+    (effects (font (size 2 2) (thickness 0.2)))
+  )
+  (gr_text "SIG B. Cu" (at 208 125.5) (layer Dwgs.User)
+    (effects (font (size 2 2) (thickness 0.2)))
+  )
+  (gr_text "SIG F. Cu" (at 208 120) (layer Dwgs.User)
+    (effects (font (size 2 2) (thickness 0.2)))
+  )
+  (gr_text "Core 1,6 mm " (at 230 123.5) (layer Dwgs.User)
+    (effects (font (size 2 2) (thickness 0.2)))
+  )
+  (gr_line (start 217 126.5) (end 242.5 126.5) (layer Dwgs.User) (width 0.2))
+  (gr_line (start 217 121) (end 242.5 121) (layer Dwgs.User) (width 0.2))
+  (gr_text "Especificaciones técnicas" (at 219.5 62.5) (layer Dwgs.User)
+    (effects (font (size 2 2) (thickness 0.2) italic))
+  )
+  (gr_text "Terminación: Estaño-Plomo(Sn/Pb)" (at 227.5 102.5) (layer Dwgs.User)
+    (effects (font (size 2 2) (thickness 0.2)))
+  )
+  (gr_text "Dist. a borde: 0,5 mm" (at 217 97.5) (layer Dwgs.User)
+    (effects (font (size 2 2) (thickness 0.2)))
+  )
+  (gr_text "0,4 mm; \n" (at 217.5 93.5) (layer Dwgs.User)
+    (effects (font (size 2 2) (thickness 0.2)))
+  )
+  (gr_text "1 mm; 0.8 mm; \n" (at 223 90.5) (layer Dwgs.User)
+    (effects (font (size 2 2) (thickness 0.2)))
+  )
+  (gr_text "Pista: 2,5 mm; 2,1 mm; \n" (at 219.5 87.5) (layer Dwgs.User)
+    (effects (font (size 2 2) (thickness 0.2)))
+  )
+  (gr_text "Margen: 0,4 mm" (at 212.5 82.5) (layer Dwgs.User)
+    (effects (font (size 2 2) (thickness 0.2)))
+  )
+  (gr_text "Vias: 1,6 mm/0,8 mm; \n    0,7 mm/0,4 mm" (at 218.5 74) (layer Dwgs.User)
+    (effects (font (size 2 2) (thickness 0.2)))
+  )
+  (gr_text "Grillas: 0,5 mm; 0,25 mm" (at 220 67.5) (layer Dwgs.User)
+    (effects (font (size 2 2) (thickness 0.2)))
+  )
+  (gr_line (start 175 71.5) (end 126 71.5) (layer Margin) (width 0.15))
+  (gr_line (start 175 120.5) (end 175 71.5) (layer Margin) (width 0.15))
+  (gr_line (start 126 120.5) (end 175 120.5) (layer Margin) (width 0.15))
+  (gr_line (start 126 71.5) (end 126 120.5) (layer Margin) (width 0.15))
+  (gr_text "ReplicaDriverPuenteHL298\nCESE2021\nIng.DamianCaputo\n" (at 151.5 76) (layer B.SilkS)
     (effects (font (size 1 1) (thickness 0.15)) (justify mirror))
   )
   (dimension 50 (width 0.15) (layer Dwgs.User)
     (gr_text "50,000 mm" (at 150.5 64.7) (layer Dwgs.User)
-      (effects (font (size 1 1) (thickness 0.15)))
+      (effects (font (size 2 2) (thickness 0.2)))
     )
     (feature1 (pts (xy 175.5 71) (xy 175.5 65.413579)))
@@
   )
   (dimension 50 (width 0.15) (layer Dwgs.User)
-    (gr_text "50,000 mm" (at 181.8 96 270) (layer Dwgs.User)
-      (effects (font (size 1 1) (thickness 0.15)))
+    (gr_text "50,000 mm" (at 181.8 96 -90) (layer Dwgs.User)
+      (effects (font (size 2 2) (thickness 0.2)))
     )
     (feature1 (pts (xy 175.5 121) (xy 181.086421 121)))
@@
     (effects (font (size 1 1) (thickness 0.15)))
   )
-  (gr_line (start 125.5 121) (end 125.5 71) (layer Edge.Cuts) (width 0.05))
-  (gr_line (start 175.5 121) (end 125.5 121) (layer Edge.Cuts) (width 0.05))
-  (gr_line (start 175.5 71) (end 175.5 121) (layer Edge.Cuts) (width 0.05))
-  (gr_line (start 125.5 71) (end 175.5 71) (layer Edge.Cuts) (width 0.05))
-  (via (at 140 88) (size 0.7) (drill 0.4) (layers F.Cu B.Cu) (net 1))
+  (gr_line (start 125.5 121) (end 125.5 71) (layer Edge.Cuts) (width 0.2))
+  (gr_line (start 175.5 121) (end 125.5 121) (layer Edge.Cuts) (width 0.2))
+  (gr_line (start 175.5 71) (end 175.5 121) (layer Edge.Cuts) (width 0.2))
+  (via (at 140 88.5) (size 0.7) (drill 0.4) (layers F.Cu B.Cu) (net 1))
   (via (at 141 91) (size 0.7) (drill 0.4) (layers F.Cu B.Cu) (net 1))
   (via (at 140 95) (size 0.7) (drill 0.4) (layers F.Cu B.Cu) (net 1))
@@
   (segment (start 146.54 98.46) (end 143.5 98.46) (width 0.8) (layer F.Cu) (net 15))
   (segment (start 150.755 94.245) (end 146.54 98.46) (width 0.8) (layer F.Cu) (net 15))
-  (zone (net 1) (net_name GND) (layer B.Cu) (hatch edge 0.508)
-    (connect_pads yes (clearance 0.508))
-    (min_thickness 0.254)
-    (fill yes (arc_segments 32) (thermal_gap 0.508) (thermal_bridge_width 0.508))
-    (polygon
-      (pts
-        (xy 175.5 121) (xy 125.5 121) (xy 125.5 71) (xy 175.5 71)
-      )
-    )
-  )
   (zone (net 1) (net_name GND) (layer F.Cu) (hatch edge 0.508)
     (connect_pads (clearance 0.508))
@@
     (polygon
       (pts
-        (xy 175.5 121) (xy 125.5 121) (xy 125.5 71) (xy 175.5 71)
+        (xy 179 125) (xy 121.5 125) (xy 121.5 67) (xy 179 67)
       )
     )
+  )
+  (zone (net 1) (net_name GND) (layer B.Cu) (hatch edge 0.508)
+    (connect_pads (clearance 0.508))
+    (min_thickness 0.254)
+    (fill yes (arc_segments 32) (thermal_gap 0.508) (thermal_bridge_width 0.508))
+    (polygon
+      (pts
+        (xy 182.5 128.5) (xy 117.5 128.5) (xy 117.5 63) (xy 182.5 63)
+      )
+    )

Commit message: Add files via upload
Other:
- board text added: "Terminación: HASL"
- board text removed: "Terminación: Estaño-Plomo(Sn/Pb)"
Changed lines of the file:
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@@
     (effects (font (size 2 2) (thickness 0.2) italic))
   )
-  (gr_text "Terminación: Estaño-Plomo(Sn/Pb)" (at 227.5 102.5) (layer Dwgs.User)
+  (gr_text "Terminación: HASL" (at 214 102.5) (layer Dwgs.User)
     (effects (font (size 2 2) (thickness 0.2)))
   )
@@
   )
   (dimension 50 (width 0.15) (layer Dwgs.User)
-    (gr_text "50,000 mm" (at 150.5 64.7) (layer Dwgs.User)
+    (gr_text "50,00 mm" (at 150.5 58.15) (layer Dwgs.User)
       (effects (font (size 2 2) (thickness 0.2)))
     )
-    (feature1 (pts (xy 175.5 71) (xy 175.5 65.413579)))
-    (feature2 (pts (xy 125.5 71) (xy 125.5 65.413579)))
-    (crossbar (pts (xy 125.5 66) (xy 175.5 66)))
-    (arrow1a (pts (xy 175.5 66) (xy 174.373496 66.586421)))
-    (arrow1b (pts (xy 175.5 66) (xy 174.373496 65.413579)))
-    (arrow2a (pts (xy 125.5 66) (xy 126.626504 66.586421)))
-    (arrow2b (pts (xy 125.5 66) (xy 126.626504 65.413579)))
+    (feature1 (pts (xy 175.5 71) (xy 175.5 59.913579)))
+    (feature2 (pts (xy 125.5 71) (xy 125.5 59.913579)))
+    (crossbar (pts (xy 125.5 60.5) (xy 175.5 60.5)))
+    (arrow1a (pts (xy 175.5 60.5) (xy 174.373496 61.086421)))
+    (arrow1b (pts (xy 175.5 60.5) (xy 174.373496 59.913579)))
+    (arrow2a (pts (xy 125.5 60.5) (xy 126.626504 61.086421)))
+    (arrow2b (pts (xy 125.5 60.5) (xy 126.626504 59.913579)))
   )
   (dimension 50 (width 0.15) (layer Dwgs.User)
-    (gr_text "50,000 mm" (at 181.8 96 -90) (layer Dwgs.User)
+    (gr_text "50,00 mm" (at 187.35 96 -90) (layer Dwgs.User)
       (effects (font (size 2 2) (thickness 0.2)))
     )
-    (feature1 (pts (xy 175.5 121) (xy 181.086421 121)))
-    (feature2 (pts (xy 175.5 71) (xy 181.086421 71)))
-    (crossbar (pts (xy 180.5 71) (xy 180.5 121)))
-    (arrow1a (pts (xy 180.5 121) (xy 179.913579 119.873496)))
-    (arrow1b (pts (xy 180.5 121) (xy 181.086421 119.873496)))
-    (arrow2a (pts (xy 180.5 71) (xy 179.913579 72.126504)))
-    (arrow2b (pts (xy 180.5 71) (xy 181.086421 72.126504)))
+    (feature1 (pts (xy 175.5 121) (xy 185.586421 121)))
+    (feature2 (pts (xy 175.5 71) (xy 185.586421 71)))
+    (crossbar (pts (xy 185 71) (xy 185 121)))
+    (arrow1a (pts (xy 185 121) (xy 184.413579 119.873496)))
+    (arrow1b (pts (xy 185 121) (xy 185.586421 119.873496)))
+    (arrow2a (pts (xy 185 71) (xy 184.413579 72.126504)))
+    (arrow2b (pts (xy 185 71) (xy 185.586421 72.126504)))
   )
   (gr_text OUT2 (at 172.5 99.25) (layer F.SilkS)
@@
   (segment (start 168.5 84) (end 171.5 81) (width 1) (layer F.Cu) (net 7))
   (segment (start 167.5 84) (end 168.5 84) (width 1) (layer F.Cu) (net 7))
-  (segment (start 160.833466 84) (end 158.59 84) (width 2.1) (layer B.Cu) (net 7))
-  (segment (start 164.70002 87.866554) (end 160.833466 84) (width 2.1) (layer B.Cu) (net 7))
-  (segment (start 158.59 84) (end 158.51 83.92) (width 2.1) (layer B.Cu) (net 7))
-  (segment (start 164.70002 87.866554) (end 164.866554 87.866554) (width 2.1) (layer B.Cu) (net 7))
-  (segment (start 170.5 93.5) (end 170.5 102.42) (width 2.1) (layer B.Cu) (net 7))
-  (segment (start 164.866554 87.866554) (end 170.5 93.5) (width 2.1) (layer B.Cu) (net 7))
+  (segment (start 160.833466 84) (end 158.59 84) (width 2.1) (layer B.Cu) (net 7) (status 1000000))
+  (segment (start 164.70002 87.866554) (end 160.833466 84) (width 2.1) (layer B.Cu) (net 7) (status 1000000))
+  (segment (start 158.59 84) (end 158.51 83.92) (width 2.1) (layer B.Cu) (net 7) (status 1000000))
+  (segment (start 164.70002 87.866554) (end 164.866554 87.866554) (width 2.1) (layer B.Cu) (net 7) (status 1000000))
+  (segment (start 170.5 93.5) (end 170.5 102.42) (width 2.1) (layer B.Cu) (net 7) (status 1000000))
+  (segment (start 164.866554 87.866554) (end 170.5 93.5) (width 2.1) (layer B.Cu) (net 7) (status 1000000))
   (segment (start 148.65 107.5) (end 148.65 103.5) (width 1) (layer F.Cu) (net 8))
   (segment (start 147.08 89) (end 147.08 104.08) (width 0.4) (layer B.Cu) (net 9))
